File: intro-to-kicad.kicad_pcb (KiCad board)
At the start: 2 copper layers, 100 x 60 mm, 20 parts, among them J1 Conn_01x01_Pin, J2 Conn_01x02_Pin, J3 Conn_01x02_Pin, U1 NE555P

Commit message: updated docs
Parts:
- removed J3: Conn_01x02_Pin, Connector_PinHeader_2.54mm:PinHeader_1x02_P2.54mm_Vertical
- added C3: 10n, Capacitor_THT:C_Disc_D3.0mm_W2.0mm_P2.50mm, F.Cu at (143.5, 83.8)
- added LS1: Speaker, Buzzer_Beeper:Buzzer_15x7.5RM7.6, F.Cu at (189.0, 83.8)
- added RV1: R_Potentiometer, Potentiometer_THT:Potentiometer_Bourns_3386F_Vertical, F.Cu at (118.5, 88.7)
- C1: footprint Capacitor_THT:C_Axial_L5.1mm_D3.1mm_P10.00mm_Horizontal -> Capacitor_THT:C_Disc_D3.8mm_W2.6mm_P2.50mm
- R1: value 10K -> 1K
- R10: value 626 -> 30K
- R11: value 650 -> 30K
- R12: value 690 -> 30K
- R13: value 730 -> 30K
- R2: value 1876 -> 30K
- R3: value 411 -> 30K
- R4: value 438 -> 30K
- R5: value 456 -> 30K
- R6: value 482 -> 30K
- R7: value 520 -> 30K
- R8: value 546 -> 30K
- R9: value 570 -> 30K
- moved J1 33.9 mm to (125.0, 78.8)
- moved U1 29.8 mm to (133.2, 76.0)
- moved C1 28.5 mm to (130.0, 78.8), turned to 90 degrees
- moved C2 12.1 mm to (173.0, 84.0)
- moved R11 9.69 mm to (178.0, 94.9), turned to -90 degrees
- moved R3 9.69 mm to (114.0, 100.0), turned to 90 degrees
- moved R10 9.65 mm to (170.0, 95.0), turned to -90 degrees
- moved R12 9.65 mm to (186.0, 95.0), turned to -90 degrees
- moved R13 9.65 mm to (194.0, 95.0), turned to -90 degrees
- moved R4 9.65 mm to (122.0, 95.0), turned to -90 degrees
- moved R5 9.65 mm to (130.0, 95.0), turned to -90 degrees
- moved R6 9.65 mm to (138.0, 95.0), turned to -90 degrees
- moved R7 9.65 mm to (146.0, 95.0), turned to -90 degrees
- moved R8 9.65 mm to (154.0, 95.0), turned to -90 degrees
- moved R9 9.65 mm to (162.0, 95.0), turned to -90 degrees
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Connections:
- R1 pad 2: +9V -> /PULL_UP
- R13 pad 2: +9V -> /KEY_12
- U1 pad 5: unconnected-(U1-CV-Pad5) -> /CV
- U2 pad 12: +9V -> /KEY_12
Routing:
- net +9V: track 149.8 -> 66.3 mm
- net /555_DIS: track 83.7 -> 64.8 mm
- net /555_Q: track 25.7 -> 42.1 mm
- net /KEY_12: track 0.00 -> 15.9 mm
- net /PULL_UP: track 0.00 -> 9.78 mm
- net /KEY_1: track 16.9 -> 26.1 mm
- net /KEY_2: track 18.1 -> 26.3 mm
- net /KEY_6: track 18.5 -> 26.1 mm
- net /KEY_5: track 18.5 -> 26.1 mm
- net /KEY_4: track 18.7 -> 26.1 mm
- net /KEY_3: track 18.8 -> 26.0 mm
- net /KEY_7: track 19.0 -> 26.1 mm
- net /KEY_8: track 19.3 -> 26.1 mm
- net /KEY_9: track 19.4 -> 26.1 mm
- net /KEY_10: track 19.4 -> 26.1 mm
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Other:
- board text added: "+9V GND"
- board text added: "STYLUS"
- board text added: "TONE ADJUSTMENT"
- board text removed: "YORK ENGINEERING SOCIETY STYLOPHONE PCB BY JACK FITTON 28/09/24"
