File: intro-to-kicad.kicad_sch (KiCad schematic)
At the start: 20 parts, among them J1 Conn_01x01_Pin, J2 Conn_01x02_Pin, J3 Conn_01x02_Pin, U1 NE555P

Commit message: updated docs
Parts:
- removed J3: Conn_01x02_Pin, Connector_PinHeader_2.54mm:PinHeader_1x02_P2.54mm_Vertical, symbol Connector:Conn_01x02_Pin
- added C3: 10n, Capacitor_THT:C_Disc_D3.0mm_W2.0mm_P2.50mm, symbol Device:C
- added LS1: Speaker, Buzzer_Beeper:Buzzer_15x7.5RM7.6, symbol Device:Speaker
- added RV1: R_Potentiometer, Potentiometer_THT:Potentiometer_Bourns_3386F_Vertical, symbol Device:R_Potentiometer
- C1: footprint Capacitor_THT:C_Axial_L5.1mm_D3.1mm_P10.00mm_Horizontal -> Capacitor_THT:C_Disc_D3.8mm_W2.6mm_P2.50mm
- R1: value 10K -> 1K
- R10: value 626 -> 30K
- R11: value 650 -> 30K
- R12: value 690 -> 30K
- R13: value 730 -> 30K
- R2: value 1876 -> 30K
- R3: value 411 -> 30K
- R4: value 438 -> 30K
- R5: value 456 -> 30K
- R6: value 482 -> 30K
- R7: value 520 -> 30K
- R8: value 546 -> 30K
- R9: value 570 -> 30K
Connections:
- net +9V: now also RV1.2; no longer R1.2, R13.2, U2.12
- net GND: now also C3.2, LS1.2
- net SPKR+: now also LS1.1
- net CV: now reaches U1.5 (CV)
- net CV: now also C3.1
- new net KEY_12: R13.2, U2.12
- new net PULL_UP: R1.2, RV1.3
Other:
- note added: "Pull up for tuning device"
- note removed: "10K Pull up to keep DIS at ~9V when stylus is not used"
- note removed: "Key 12 doesnt need its own label as its on the same wire as +9V which is a global label"
- note removed: "This pin with the X is a Non-Connect This tells the software you are intentionally not connecting this pin to anything. press Q for a NC"
- moved on the sheet: R1
