File: intro-to-kicad.kicad_sch (KiCad schematic)
At the start: 20 parts, among them J1 Conn_01x01_Pin, J2 Conn_01x02_Pin, J3 Conn_01x02_Pin, U1 NE555P

Commit message: finalised project
Parts:
- R10: value 626 -> 30K
- R11: value 650 -> 30K
- R12: value 690 -> 30K
- R13: value 730 -> 30K
- R2: value 1876 -> 30K
- R3: value 411 -> 30K
- R4: value 438 -> 30K
- R5: value 456 -> 30k
- R6: value 482 -> 30k
- R7: value 520 -> 30K
- R8: value 546 -> 30K
- R9: value 570 -> 30K
Connections:
- net +9V: no longer R13.2, U2.12
- new net KEY_12: R13.2, U2.12
Other:
- note removed: "Key 12 doesnt need its own label as its on the same wire as +9V which is a global label"
Changed lines of the file:
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@@
 		(color 0 0 0 0)
 	)
-	(junction
-		(at 41.91 104.14)
-		(diameter 0)
-		(color 0 0 0 0)
-	)
 	(no_connect
 		(at 190.5 66.04)
@@
 	(wire
 		(pts
-			(xy 39.37 104.14) (xy 41.91 104.14)
-		)
-		(stroke
-			(width 0)
-			(type default)
-		)
-	)
-	(wire
-		(pts
 			(xy 133.35 127) (xy 133.35 124.46)
 		)
@@
 		)
 	)
-	(text_box "Component Values\n\nR1 = 10 kΩ\nR2 = 1876Ω\nR3 = 411Ω\nR4 = 438Ω\nR5 = 456Ω\nR6 = 482Ω\nR7 = 520Ω\nR8 = 546Ω\nR9 = 570Ω\nR10 = 626Ω\nR11 = 650Ω\nR12 = 690Ω\nR13 = 730Ω\n\nC1 = 100 nF, ceramic\nC2 = 10 mF x 10V, electrolytic (CHECK POLARITY!)\nJ3 = speaker with impedance of eight ohms"
-		(exclude_from_sim no)
-		(at 17.78 151.13 0)
-		(size 46.99 41.91)
-		(stroke
-			(width 0)
-			(type default)
-		)
-		(fill
-			(type none)
-		)
-		(effects
-			(font
-				(face "Open Sans")
-				(size 1.27 1.27)
-			)
-			(justify left top)
-		)
-	)
 	(text "Stylus"
 		(exclude_from_sim no)
@@
 		)
 	)
-	(text "Key 12 doesnt need its\n own label as its\non the same wire as \n+9V which is a global label"
-		(exclude_from_sim no)
-		(at 46.736 133.096 0)
-		(effects
-			(font
-				(size 1.27 1.27)
-			)
-		)
-	)
 	(text "This pin with the X is a Non-Connect\nThis tells the software you are intentionally not connecting\nthis pin to anything. press Q for a NC"
 		(exclude_from_sim no)
@@
 		)
 	)
+	(label "KEY_12"
+		(at 41.91 127 0)
+		(fields_autoplaced yes)
+		(effects
+			(font
+				(size 1.27 1.27)
+			)
+			(justify left bottom)
+		)
+	)
 	(label "KEY_3"
 		(at 143.51 123.19 0)
@@
 	)
 	(symbol
-		(lib_id "power:+9V")
-		(at 39.37 104.14 90)
-		(unit 1)
-		(exclude_from_sim no)
-		(in_bom yes)
-		(on_board yes)
-		(dnp no)
-		(fields_autoplaced yes)
-		(property "Reference" "#PWR05"
-			(at 43.18 104.14 0)
-			(effects
-				(font
-					(size 1.27 1.27)
-				)
-				(hide yes)
-			)
-		)
-		(property "Value" "+9V"
-			(at 35.56 104.1399 90)
-			(effects
-				(font
-					(size 1.27 1.27)
-				)
-				(justify left)
-			)
-		)
-		(property "Footprint" ""
-			(at 39.37 104.14 0)
-			(effects
-				(font
-					(size 1.27 1.27)
-				)
-				(hide yes)
-			)
-		)
-		(property "Datasheet" ""
-			(at 39.37 104.14 0)
-			(effects
-				(font
-					(size 1.27 1.27)
-				)
-				(hide yes)
-			)
-		)
-		(property "Description" "Power symbol creates a global label with name \"+9V\""
-			(at 39.37 104.14 0)
-			(effects
-				(font
-					(size 1.27 1.27)
-				)
-				(hide yes)
-			)
-		)
-		(pin "1"
-		)
-		(instances
-			(project "intro-to-kicad"
-				(path "/a4345fa4-d9e0-4460-8734-083d5039e811"
-					(reference "#PWR05")
-					(unit 1)
-				)
-			)
-		)
-	)
-	(symbol
 		(lib_id "power:PWR_FLAG")
 		(at 76.2 63.5 0)
@@
 			)
 		)
-		(property "Value" "730"
+		(property "Value" "30K"
 			(at 49.53 100.33 90)
 			(effects
@@
 			)
 		)
-		(property "Value" "482"
+		(property "Value" "30k"
 			(at 132.08 100.33 90)
 			(effects
@@
 			)
 		)
-		(property "Value" "1876"
+		(property "Value" "30K"
 			(at 179.07 100.33 90)
 			(effects
@@
 			)
 		)
-		(property "Value" "690"
+		(property "Value" "30K"
 			(at 60.96 100.33 90)
 			(effects
@@
 			)
 		)
-		(property "Value" "520"
+		(property "Value" "30K"
 			(at 120.65 100.33 90)
 			(effects
@@
 			)
 		)
-		(property "Value" "650"
+		(property "Value" "30K"
 			(at 72.39 100.33 90)
 			(effects
@@
 			)
 		)
-		(property "Value" "570"
+		(property "Value" "30K"
 			(at 97.79 100.33 90)
 			(effects
@@
 			)
 		)
-		(property "Value" "626"
+		(property "Value" "30K"
 			(at 85.09 100.33 90)
 			(effects
@@
 			)
 		)
-		(property "Value" "411"
+		(property "Value" "30K"
 			(at 167.64 100.33 90)
 			(effects
@@
 			)
 		)
-		(property "Value" "546"
+		(property "Value" "30K"
 			(at 109.22 100.33 90)
 			(effects
@@
 			)
 		)
-		(property "Value" "438"
+		(property "Value" "30K"
 			(at 156.21 100.33 90)
 			(effects
@@
 			)
 		)
-		(property "Value" "456"
+		(property "Value" "30k"
 			(at 144.78 100.33 90)
 			(effects
